File: tt-eom-driver/tt-eom-driver.kicad_sch (KiCad schematic)
At the start: 51 parts, among them IC1 VCA820ID, IC2 VCA820ID, J1 Conn_Coaxial, J2 Conn_Coaxial, U1 THS3491xDDA, U2 THS3491xDDA, U3 PAT1220-C-1DB, U4 PAT1220-C-1DB, U5 SBTCJ-13-75+

Commit message: added pwr supply
Parts:
- added C14: 0.8p, symbol Device:C
- added C23, C27: 6.8u, Capacitor_SMD:C_0603_1608Metric, symbol Device:C
- added C24, C28: 2.2u, Capacitor_SMD:C_0603_1608Metric, symbol Device:C
- added C25, C29: 0.1u, Capacitor_SMD:C_0603_1608Metric, symbol Device:C
- added C26, C30: 100p, Capacitor_SMD:C_0603_1608Metric, symbol Device:C
- added C31: 0.1u, symbol Device:C
- added C32: 0.22u, symbol Device:C
- added C33, C34: 1u, symbol Device:C
- added C35: 1n, symbol Device:C
- added C36: 100p, symbol Device:C
- added IC3: DAC7562SDGST, SOP50P490X110-10N, symbol DAC7562SDGST:DAC7562SDGST
- added J3, J4: Conn_Coaxial, symbol Connector:Conn_Coaxial
- added L1: 3.6n, symbol Device:L
- added R21: 43.3, symbol Device:R
- added R22: 86.6, symbol Device:R
- added R23, R24: 49.9, symbol Device:R
- added R25: 4.99, symbol Device:R
- added R26, R27: 1M, symbol Device:R
- added R28, R29, R30: 33, symbol Device:R
- added R31, R34: 10k, symbol Device:R
- added R32, R33: 1k, symbol Device:R
- R19, R20: value 49.9 -> 0
Connections:
- net COUP: now also R21.2
- net FOSTER_IN: now also J3.1 (In)
- net GND: now also C14.1, C23.1, C24.1, C25.1, C26.1, C27.1, C28.1, C29.1, C30.1, C31.1, C32.2, C33.1, C34.1, C35.1, C36.1, IC3.3 (GND), IC3.4 (~{LDAC}), J3.2 (Ext), J4.2 (Ext), R22.2, R23.2, R24.2, R26.2, R27.2; no longer IC1.6 (-VIN), IC2.6 (-VIN)
- net THS_OUT_T1: now also R25.2; no longer U5.1 (PORT_1_(180°)_)
- net THS_OUT_T2: now also L1.2; no longer U5.3 (PORT_2_(0°)_)
- net VG1: now also C33.2, R27.1, R32.2
- net VG2: now also C34.2, R26.1, R33.2
- net +15V renamed +15V1
- net +15V1: no longer U2.7 (V+), U2.8 (~{PD})
- net -15V renamed -15V1
- net -15V1: no longer U2.4 (V-)
- new net: IC2.6 (-VIN), R23.1
- new net: C32.1, IC3.10 (VREFIN/VREFOUT)
- new net: IC1.6 (-VIN), R24.1
- new net: C14.2, L1.1, U5.3 (PORT_2_(0°)_)
- new net: IC3.5 (~{CLR}), R31.2
- new net: R25.1, U5.1 (PORT_1_(180°)_)
- new net: IC3.6 (~{SYNC}), R28.1, R34.2
- new net: IC3.7 (SCLK), R29.1
- new net: IC3.8 (DIN), R30.1
- new net +15V2: C23.2, C24.2, C25.2, C26.2, U2.7 (V+), U2.8 (~{PD})
- new net +3.3V: C31.2, C35.2, C36.2, IC3.9 (AVDD), R31.1, R34.1
- new net -15V2: C27.2, C28.2, C29.2, C30.2, U2.4 (V-)
- new net COUP_ADC: J4.1 (In), R21.1, R22.1
- new net SCLK1: R29.2
- new net SDI1: R30.2
- new net SYNC1: R28.2
- new net VG1_un: IC3.1 (VOUTA), R32.1
- new net VG2_un: IC3.2 (VOUTB), R33.1
Other:
- added sheet sch1 (sch1.kicad_sch)
- note added: "75 ohm 180 hybrid"
- note added: "75 ohm coupler"
- note added: "75->50 ohm match (for ADC)"
- note added: "DAC filters"
- note added: "FOSTER (75 ohm) ADC (50 ohm)"
- note added: "Outputs"
- moved on the sheet: HY1, R15

Commit message: little error to DAC
Parts:
- removed C3, C7: 0.1u, Capacitor_SMD:C_0603_1608Metric, symbol Device:C
- removed R12, R16: 220, symbol Device:R
- added C57, C58: 0.1u, Capacitor_SMD:C_0603_1608Metric, symbol Device:C
Connections:
- net +15V1: now also C57.2
- net +15V2: now also C58.2
- net -15V1: now also C57.1
- net -15V2: now also C58.1
